File: Плата управления/Temperture_measure.kicad_sch (KiCad schematic)
At the start: 3 parts

Commit message: Добавил все документы
Parts:
- renumbered R21 to R17, R22 to R18, R23 to R19
Changed lines of the file:
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@@
   (symbol (lib_id "Device:R_Small") (at 148.59 97.155 180) (unit 1)
     (in_bom yes) (on_board yes) (dnp no) (fields_autoplaced)
-    (property "Reference" "R23" (at 151.13 96.52 0)
+    (property "Reference" "R19" (at 151.13 96.52 0)
       (effects (font (size 1.27 1.27)) (justify right))
     )
@@
       (project "Плата управления"
         (path "/75f4c67c-bbde-4446-8f82-67797a1b269f/d6b8b9ce-300b-4d22-9d4c-9182eba581b1"
-          (reference "R23") (unit 1)
+          (reference "R19") (unit 1)
         )
         (path "/75f4c67c-bbde-4446-8f82-67797a1b269f/c91ff3ec-ad20-4326-acd4-2c9dea437172"
@@
   (symbol (lib_id "power:+3.3V") (at 139.7 92.075 0) (unit 1)
     (in_bom yes) (on_board yes) (dnp no) (fields_autoplaced)
-    (property "Reference" "#PWR029" (at 139.7 95.885 0)
+    (property "Reference" "#PWR026" (at 139.7 95.885 0)
       (effects (font (size 1.27 1.27)) hide)
     )
@@
       (project "Плата управления"
         (path "/75f4c67c-bbde-4446-8f82-67797a1b269f/d6b8b9ce-300b-4d22-9d4c-9182eba581b1"
-          (reference "#PWR029") (unit 1)
+          (reference "#PWR026") (unit 1)
         )
       )
@@
   (symbol (lib_id "Device:R_Small") (at 130.81 97.155 180) (unit 1)
     (in_bom yes) (on_board yes) (dnp no) (fields_autoplaced)
-    (property "Reference" "R21" (at 133.35 96.52 0)
+    (property "Reference" "R17" (at 133.35 96.52 0)
       (effects (font (size 1.27 1.27)) (justify right))
     )
@@
       (project "Плата управления"
         (path "/75f4c67c-bbde-4446-8f82-67797a1b269f/d6b8b9ce-300b-4d22-9d4c-9182eba581b1"
-          (reference "R21") (unit 1)
+          (reference "R17") (unit 1)
         )
         (path "/75f4c67c-bbde-4446-8f82-67797a1b269f/c91ff3ec-ad20-4326-acd4-2c9dea437172"
@@
   (symbol (lib_id "Device:R_Small") (at 139.7 97.155 180) (unit 1)
     (in_bom yes) (on_board yes) (dnp no) (fields_autoplaced)
-    (property "Reference" "R22" (at 142.24 96.52 0)
+    (property "Reference" "R18" (at 142.24 96.52 0)
       (effects (font (size 1.27 1.27)) (justify right))
     )
@@
       (project "Плата управления"
         (path "/75f4c67c-bbde-4446-8f82-67797a1b269f/d6b8b9ce-300b-4d22-9d4c-9182eba581b1"
-          (reference "R22") (unit 1)
+          (reference "R18") (unit 1)
         )
         (path "/75f4c67c-bbde-4446-8f82-67797a1b269f/c91ff3ec-ad20-4326-acd4-2c9dea437172"
