File: Плата управления/SWD.kicad_sch (KiCad schematic)
At the start: 2 parts, among them J8 SWD

Commit message: Добавил документы
Other:
- note added: "SWD"
- moved on the sheet: D6, J8
Changed lines of the file:
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@@
 (kicad_sch (version 20230121) (generator eeschema)
   (paper "A4")
-  (wire (pts (xy 92.71 88.9) (xy 92.71 90.17))
+  (title_block
+    (comment 1 "МПСТ.76721.758764.02.Э3.М")
+  )
+  (wire (pts (xy 158.115 93.98) (xy 158.115 95.25))
     (stroke (width 0) (type default))
   )
-  (wire (pts (xy 92.71 105.41) (xy 92.71 106.68))
+  (wire (pts (xy 158.115 110.49) (xy 158.115 111.76))
     (stroke (width 0) (type default))
   )
-  (wire (pts (xy 91.44 105.41) (xy 92.71 105.41))
+  (wire (pts (xy 156.845 110.49) (xy 158.115 110.49))
     (stroke (width 0) (type default))
   )
-  (wire (pts (xy 91.44 97.79) (xy 92.71 97.79))
+  (wire (pts (xy 156.845 102.87) (xy 158.115 102.87))
     (stroke (width 0) (type default))
   )
-  (wire (pts (xy 92.71 97.79) (xy 92.71 95.25))
+  (wire (pts (xy 158.115 102.87) (xy 158.115 100.33))
     (stroke (width 0) (type default))
   )
-  (global_label "SWCLK" (shape input) (at 91.44 102.87 0) (fields_autoplaced)
+  (rectangle (start 140.97 79.375) (end 171.45 123.19)
+    (stroke (width 0) (type dash))
+    (fill (type none))
+  )
+  (text "SWD" (at 153.035 78.105 0)
+    (effects (font (size 2 2) bold) (justify left bottom))
+  )
+  (global_label "SWCLK" (shape input) (at 156.845 107.95 0) (fields_autoplaced)
     (effects (font (size 1.27 1.27)) (justify left))
-    (property "Intersheetrefs" "${INTERSHEET_REFS}" (at 100.6542 102.87 0)
+    (property "Intersheetrefs" "${INTERSHEET_REFS}" (at 166.0592 107.95 0)
       (effects (font (size 1.27 1.27)) (justify left) hide)
     )
   )
-  (global_label "SWDIO" (shape input) (at 91.44 100.33 0) (fields_autoplaced)
+  (global_label "SWDIO" (shape input) (at 156.845 105.41 0) (fields_autoplaced)
     (effects (font (size 1.27 1.27)) (justify left))
-    (property "Intersheetrefs" "${INTERSHEET_REFS}" (at 100.2914 100.33 0)
+    (property "Intersheetrefs" "${INTERSHEET_REFS}" (at 165.6964 105.41 0)
       (effects (font (size 1.27 1.27)) (justify left) hide)
     )
   )
-  (symbol (lib_id "power:+3.3V") (at 92.71 88.9 0) (unit 1)
+  (symbol (lib_id "power:+3.3V") (at 158.115 93.98 0) (unit 1)
     (in_bom yes) (on_board yes) (dnp no) (fields_autoplaced)
-    (property "Reference" "#PWR070" (at 92.71 92.71 0)
+    (property "Reference" "#PWR070" (at 158.115 97.79 0)
       (effects (font (size 1.27 1.27)) hide)
     )
-    (property "Value" "+3.3V" (at 92.71 83.82 0)
+    (property "Value" "+3.3V" (at 158.115 88.9 0)
       (effects (font (size 1.27 1.27)))
     )
-    (property "Footprint" "" (at 92.71 88.9 0)
+    (property "Footprint" "" (at 158.115 93.98 0)
       (effects (font (size 1.27 1.27)) hide)
     )
-    (property "Datasheet" "" (at 92.71 88.9 0)
+    (property "Datasheet" "" (at 158.115 93.98 0)
       (effects (font (size 1.27 1.27)) hide)
     )
@@
     )
   )
-  (symbol (lib_id "power:GND") (at 92.71 106.68 0) (unit 1)
+  (symbol (lib_id "power:GND") (at 158.115 111.76 0) (unit 1)
     (in_bom yes) (on_board yes) (dnp no) (fields_autoplaced)
-    (property "Reference" "#PWR071" (at 92.71 113.03 0)
+    (property "Reference" "#PWR071" (at 158.115 118.11 0)
       (effects (font (size 1.27 1.27)) hide)
     )
-    (property "Value" "GND" (at 92.71 111.76 0)
+    (property "Value" "GND" (at 158.115 116.84 0)
       (effects (font (size 1.27 1.27)))
     )
-    (property "Footprint" "" (at 92.71 106.68 0)
+    (property "Footprint" "" (at 158.115 111.76 0)
       (effects (font (size 1.27 1.27)) hide)
     )
-    (property "Datasheet" "" (at 92.71 106.68 0)
+    (property "Datasheet" "" (at 158.115 111.76 0)
       (effects (font (size 1.27 1.27)) hide)
     )
@@
     )
   )
-  (symbol (lib_id "Connector_Generic:Conn_01x04") (at 86.36 102.87 180) (unit 1)
-    (in_bom yes) (on_board yes) (dnp no) (fields_autoplaced)
-    (property "Reference" "J8" (at 86.36 91.44 0)
+  (symbol (lib_id "Connector_Generic:Conn_01x04") (at 151.765 107.95 180) (unit 1)
+    (in_bom yes) (on_board yes) (dnp no)
+    (property "Reference" "J8" (at 151.765 100.33 0)
       (effects (font (size 1.27 1.27)))
     )
-    (property "Value" "SWD" (at 86.36 93.98 0)
+    (property "Value" "SWD" (at 149.225 106.68 90)
       (effects (font (size 1.27 1.27)))
     )
-    (property "Footprint" "Connector_PinHeader_2.54mm:PinHeader_1x04_P2.54mm_Vertical" (at 86.36 102.87 0)
+    (property "Footprint" "Connector_PinHeader_2.54mm:PinHeader_1x04_P2.54mm_Vertical" (at 151.765 107.95 0)
       (effects (font (size 1.27 1.27)) hide)
     )
-    (property "Datasheet" "~" (at 86.36 102.87 0)
+    (property "Datasheet" "~" (at 151.765 107.95 0)
       (effects (font (size 1.27 1.27)) hide)
     )
@@
     )
   )
-  (symbol (lib_id "Device:D_Small") (at 92.71 92.71 270) (unit 1)
-    (in_bom yes) (on_board yes) (dnp no) (fields_autoplaced)
-    (property "Reference" "D6" (at 95.25 91.44 90)
+  (symbol (lib_id "Device:D_Small") (at 158.115 97.79 270) (unit 1)
+    (in_bom yes) (on_board yes) (dnp no)
+    (property "Reference" "D6" (at 160.02 97.79 90)
       (effects (font (size 1.27 1.27)) (justify left))
     )
-    (property "Value" "D_Small" (at 95.25 93.98 90)
+    (property "Value" "D_Small" (at 160.655 99.06 90)
       (effects (font (size 1.27 1.27)) (justify left) hide)
     )
-    (property "Footprint" "Diode_SMD:D_SOD-323_HandSoldering" (at 92.71 92.71 90)
+    (property "Footprint" "Diode_SMD:D_SOD-323_HandSoldering" (at 158.115 97.79 90)
       (effects (font (size 1.27 1.27)) hide)
     )
-    (property "Datasheet" "~" (at 92.71 92.71 90)
+    (property "Datasheet" "~" (at 158.115 97.79 90)
       (effects (font (size 1.27 1.27)) hide)
     )
-    (property "Sim.Device" "D" (at 92.71 92.71 0)
+    (property "Sim.Device" "D" (at 158.115 97.79 0)
       (effects (font (size 1.27 1.27)) hide)
     )
-    (property "Sim.Pins" "1=K 2=A" (at 92.71 92.71 0)
+    (property "Sim.Pins" "1=K 2=A" (at 158.115 97.79 0)
       (effects (font (size 1.27 1.27)) hide)
     )

Commit message: Добавил все документы
Parts:
- renumbered D6 to D13, J8 to J10
Changed lines of the file:
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@@
   (symbol (lib_id "power:+3.3V") (at 158.115 93.98 0) (unit 1)
     (in_bom yes) (on_board yes) (dnp no) (fields_autoplaced)
-    (property "Reference" "#PWR070" (at 158.115 97.79 0)
+    (property "Reference" "#PWR0105" (at 158.115 97.79 0)
       (effects (font (size 1.27 1.27)) hide)
     )
@@
       (project "Плата управления"
         (path "/75f4c67c-bbde-4446-8f82-67797a1b269f/47f4c3e6-ca16-48bd-a07f-b1f138b5b42e"
-          (reference "#PWR070") (unit 1)
+          (reference "#PWR0105") (unit 1)
         )
       )
@@
   (symbol (lib_id "power:GND") (at 158.115 111.76 0) (unit 1)
     (in_bom yes) (on_board yes) (dnp no) (fields_autoplaced)
-    (property "Reference" "#PWR071" (at 158.115 118.11 0)
+    (property "Reference" "#PWR0106" (at 158.115 118.11 0)
       (effects (font (size 1.27 1.27)) hide)
     )
@@
       (project "Плата управления"
         (path "/75f4c67c-bbde-4446-8f82-67797a1b269f/47f4c3e6-ca16-48bd-a07f-b1f138b5b42e"
-          (reference "#PWR071") (unit 1)
+          (reference "#PWR0106") (unit 1)
         )
       )
@@
   (symbol (lib_id "Connector_Generic:Conn_01x04") (at 151.765 107.95 180) (unit 1)
     (in_bom yes) (on_board yes) (dnp no)
-    (property "Reference" "J8" (at 151.765 100.33 0)
+    (property "Reference" "J10" (at 151.765 100.33 0)
       (effects (font (size 1.27 1.27)))
     )
@@
       (project "Плата управления"
         (path "/75f4c67c-bbde-4446-8f82-67797a1b269f/47f4c3e6-ca16-48bd-a07f-b1f138b5b42e"
-          (reference "J8") (unit 1)
+          (reference "J10") (unit 1)
         )
       )
@@
   (symbol (lib_id "Device:D_Small") (at 158.115 97.79 270) (unit 1)
     (in_bom yes) (on_board yes) (dnp no)
-    (property "Reference" "D6" (at 160.02 97.79 90)
+    (property "Reference" "D13" (at 160.02 97.79 90)
       (effects (font (size 1.27 1.27)) (justify left))
     )
@@
       (project "Плата управления"
         (path "/75f4c67c-bbde-4446-8f82-67797a1b269f/47f4c3e6-ca16-48bd-a07f-b1f138b5b42e"
-          (reference "D6") (unit 1)
+          (reference "D13") (unit 1)
         )
       )

Commit message: Версия под отчёт
Changed lines of the file:
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@@
   )
   (text "SWD" (at 153.035 78.105 0)
-    (effects (font (size 2 2) bold) (justify left bottom))
+    (effects (font (size 2.5 2.5) bold) (justify left bottom))
   )
   (global_label "SWCLK" (shape input) (at 156.845 107.95 0) (fields_autoplaced)
@@
           (reference "#PWR0105") (unit 1)
         )
+        (path "/75f4c67c-bbde-4446-8f82-67797a1b269f/a1fd62e4-a3fa-422c-840b-ff6e9353e9fd"
+          (reference "#PWR0110") (unit 1)
+        )
       )
     )
@@
         (path "/75f4c67c-bbde-4446-8f82-67797a1b269f/47f4c3e6-ca16-48bd-a07f-b1f138b5b42e"
           (reference "#PWR0106") (unit 1)
+        )
+        (path "/75f4c67c-bbde-4446-8f82-67797a1b269f/a1fd62e4-a3fa-422c-840b-ff6e9353e9fd"
+          (reference "#PWR0111") (unit 1)
         )
       )
@@
         (path "/75f4c67c-bbde-4446-8f82-67797a1b269f/47f4c3e6-ca16-48bd-a07f-b1f138b5b42e"
           (reference "J10") (unit 1)
+        )
+        (path "/75f4c67c-bbde-4446-8f82-67797a1b269f/a1fd62e4-a3fa-422c-840b-ff6e9353e9fd"
+          (reference "J11") (unit 1)
         )
       )
@@
           (reference "D13") (unit 1)
         )
+        (path "/75f4c67c-bbde-4446-8f82-67797a1b269f/a1fd62e4-a3fa-422c-840b-ff6e9353e9fd"
+          (reference "D16") (unit 1)
+        )
       )
