File: Плата управления/Overcurrent_Protection.kicad_sch (KiCad schematic)
At the start: 10 parts, among them U5 INA283, U5 LMV7239M5

Commit message: Поправил посадочное место LMV7239M5
Parts:
- U5: footprint Package_TO_SOT_SMD:SOT-353_SC-70-5 -> Package_TO_SOT_SMD:SOT-23-5_HandSoldering
Changed lines of the file:
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@@
       (effects (font (size 1.27 1.27)))
     )
-    (property "Footprint" "Package_TO_SOT_SMD:SOT-353_SC-70-5" (at 169.545 113.03 0)
+    (property "Footprint" "Package_TO_SOT_SMD:SOT-23-5_HandSoldering" (at 169.545 113.03 0)
       (effects (font (size 1.27 1.27)) (justify left) hide)
     )
