File: Плата управления/Power_Supply.kicad_sch (KiCad schematic)
At the start: 21 parts, among them U10 LMV321, U11 LM2594HVM-12, U9 LM2594HVM-12

Commit message: Поправил посадочное место LMV321
Parts:
- U10: footprint Package_TO_SOT_SMD:SOT-23-5_HandSoldering -> Package_TO_SOT_SMD:SOT-353_SC-70-5_Handsoldering
Changed lines of the file:
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@@
       (effects (font (size 1.27 1.27)))
     )
-    (property "Footprint" "Package_TO_SOT_SMD:SOT-23-5_HandSoldering" (at 208.915 70.485 0)
+    (property "Footprint" "Package_TO_SOT_SMD:SOT-353_SC-70-5_Handsoldering" (at 208.915 70.485 0)
       (effects (font (size 1.27 1.27)) (justify left) hide)
     )
