File: Плата управления/Power_Supply.kicad_sch (KiCad schematic)
At the start: 21 parts, among them U10 LM2594HVM-12, U12 LM2594HVM-12, U3 LMV321

Commit message: Добавил все документы
Parts:
- renumbered C12 to C33, C20 to C34, C42 to C35, C25 to C36, C36 to C37, C37 to C38, C45 to C39, C41 to C40, C44 to C41, C43 to C42, C18 to C43, D5 to D7, D4 to D8, R14 to R32, R20 to R33, R15 to R34, U3 to U10, U12 to U11, U10 to U9
Connections:
- net +24V: now also C34.1, C35.1, U9.7 (VIN)

Commit message: Версия под отчёт
Changed lines of the file:
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@@
   )
   (text "Питание 3.3В" (at 97.79 111.125 0)
-    (effects (font (size 2 2) (thickness 0.4) bold) (justify left bottom))
+    (effects (font (size 2.5 2.5) (thickness 0.4) bold) (justify left bottom))
   )
   (text "Измерение напряжения ЗПТ" (at 185.42 34.29 0)
-    (effects (font (size 2 2) (thickness 0.4) bold) (justify left bottom))
+    (effects (font (size 2.5 2.5) (thickness 0.4) bold) (justify left bottom))
   )
   (text "Питание 12В" (at 98.425 34.29 0)
-    (effects (font (size 2 2) (thickness 0.4) bold) (justify left bottom))
+    (effects (font (size 2.5 2.5) (thickness 0.4) bold) (justify left bottom))
   )
   (global_label "DC_Voltage_MCU" (shape output) (at 230.505 70.485 0) (fields_autoplaced)

Commit message: VER2.0
Parts:
- removed C36, C39, C40: 10u, Capacitor_SMD:C_1210_3225Metric_Pad1.33x2.70mm_HandSolder, symbol Device:C_Small
- removed C42, C43: 100u, Capacitor_SMD:C_1206_3216Metric_Pad1.33x1.80mm_HandSolder, symbol Device:C_Small
- added C32: 330u, Capacitor_Tantalum_SMD:CP_EIA-7343-31_Kemet-D_Pad2.25x2.55mm_HandSolder, symbol Device:C_Polarized_Small_US
- added C36, C39: 100u, Capacitor_Tantalum_SMD:CP_EIA-7343-31_Kemet-D_Pad2.25x2.55mm_HandSolder, symbol Device:C_Polarized_Small_US
- L1: value 33u -> 47u; footprint Inductor_SMD:L_Vishay_IHLP-2525 -> Capacitor_SMD:C_2220_5650Metric_Pad1.97x5.40mm_HandSolder
- L2: value 22u -> 47u; footprint Inductor_SMD:L_Vishay_IHLP-2525 -> Capacitor_SMD:C_2220_5650Metric_Pad1.97x5.40mm_HandSolder
- U10: footprint Package_TO_SOT_SMD:SOT-23-5_HandSoldering -> Package_TO_SOT_SMD:SOT-353_SC-70-5_Handsoldering
Connections:
- net +12V: now also C36.1, C39.1
- net +3.3V: now also C32.1
- net GND: now also C32.2, C36.2, C39.2

Commit message: Новые драйвера и разъёмы
Parts:
- added C53, C55: 10u, Capacitor_SMD:C_1210_3225Metric_Pad1.33x2.70mm_HandSolder, symbol Device:C_Small
Connections:
- net +24V: now also C53.1, C55.1
- net GND: now also C53.2, C55.2
Other:
- moved on the sheet: C34

Commit message: Добавил все в BOM
Parts:
- C36, C39: footprint Capacitor_Tantalum_SMD:CP_EIA-7343-31_Kemet-D_Pad2.25x2.55mm_HandSolder -> Capacitor_Tantalum_SMD:CP_EIA-7343-43_Kemet-X_Pad2.25x2.55mm_HandSolder
- U10: footprint Package_TO_SOT_SMD:SOT-353_SC-70-5_Handsoldering -> Package_TO_SOT_SMD:SOT-23-5_HandSoldering
Changed lines of the file:
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@@
 			)
 		)
-		(property "Footprint" "Capacitor_Tantalum_SMD:CP_EIA-7343-31_Kemet-D_Pad2.25x2.55mm_HandSolder"
+		(property "Footprint" "Capacitor_Tantalum_SMD:CP_EIA-7343-43_Kemet-X_Pad2.25x2.55mm_HandSolder"
 			(at 84.455 148.59 0)
 			(effects
@@
 			)
 		)
-		(property "Description" ""
+		(property "Description" "CA45-E025K107T"
 			(at 84.455 148.59 0)
 			(effects
@@
 			)
 		)
-		(property "Footprint" "Package_TO_SOT_SMD:SOT-353_SC-70-5_Handsoldering"
+		(property "Footprint" "Package_TO_SOT_SMD:SOT-23-5_HandSoldering"
 			(at 208.915 70.485 0)
 			(effects
@@
 			)
 		)
-		(property "Footprint" "Capacitor_Tantalum_SMD:CP_EIA-7343-31_Kemet-D_Pad2.25x2.55mm_HandSolder"
+		(property "Footprint" "Capacitor_Tantalum_SMD:CP_EIA-7343-43_Kemet-X_Pad2.25x2.55mm_HandSolder"
 			(at 132.08 71.12 0)
 			(effects
@@
 			)
 		)
-		(property "Description" ""
+		(property "Description" "CA45-E025K107T"
 			(at 132.08 71.12 0)
 			(effects
