File: Плата управления/Плата управления.kicad_sch (KiCad schematic)
At the start: 0 parts

Commit message: VER2.0
Other:
- removed sheet RS485
Changed lines of the file:
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@@
-    )
-  )
-  (sheet (at 29.21 105.41) (size 52.07 33.02) (fields_autoplaced)
-    (stroke (width 0.1524) (type solid))
-    (fill (color 0 0 0 0.0000))
-    (property "Sheetname" "RS485" (at 29.21 104.0834 0)
-      (effects (font (size 2.5 2.5)) (justify left bottom))
-    )
-    (property "Sheetfile" "RS485.kicad_sch" (at 29.21 139.0146 0)
-      (effects (font (size 1.27 1.27)) (justify left top) hide)
-    )
-    (property "Поле2" "" (at 29.21 105.41 0)
-      (effects (font (size 1.27 1.27)) hide)
-    )
-    (instances
-      (project "Плата управления"
-        (path "/75f4c67c-bbde-4446-8f82-67797a1b269f" (page "10"))
-      )
     )
   )
