File: Плата управления/Driver.kicad_sch (KiCad schematic)
At the start: 25 parts

Commit message: Привел в порядок схему
Other:
- note added: "Драйвер А"
- note added: "Драйвер В"
- note added: "Драйвер С"
- moved on the sheet: C1, C2, C3, C4, C5, C6, D1, D2, D3, D4, D5, D6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

Commit message: Ещё нужно доработать
Parts:
- removed C5: 10u, Capacitor_SMD:C_0603_1608Metric_Pad1.08x0.95mm_HandSolder, symbol Device:C_Small
- removed C6: BS, Capacitor_SMD:C_0805_2012Metric_Pad1.18x1.45mm_HandSolder, symbol Device:C_Small
- removed D2, D4, D6: ADP3110A, Package_DFN_QFN:DFN-8-1EP_3x3mm_P0.65mm_EP1.7x2.05mm, symbol IGBT_MOSFET_Drivers:ADP3110A
- removed D5: D_Small, Diode_SMD:D_SOD-323, symbol Device:D_Small
- removed R10, R11: 2.7, Resistor_SMD:R_0805_2012Metric_Pad1.20x1.40mm_HandSolder, symbol Device:R_Small
- removed R12, R13: 10k, Resistor_SMD:R_0603_1608Metric_Pad0.98x0.95mm_HandSolder, symbol Device:R_Small
- added C14: 10u, Capacitor_SMD:C_0603_1608Metric_Pad1.08x0.95mm_HandSolder, symbol Device:C_Small
- added C15: BS, Capacitor_SMD:C_0805_2012Metric_Pad1.18x1.45mm_HandSolder, symbol Device:C_Small
- added D2: D_Small, Diode_SMD:D_SOD-323, symbol Device:D_Small
- added R27: 2.7, Resistor_SMD:R_0805_2012Metric_Pad1.20x1.40mm_HandSolder, symbol Device:R_Small
- added R28, R32: 10k, Resistor_SMD:R_0603_1608Metric_Pad0.98x0.95mm_HandSolder, symbol Device:R_Small
- added U11, U4, U9: IR2184, Package_SO:SO-8_3.9x4.9mm_P1.27mm, symbol Driver_FET:IR2184
- R1: value 10k -> 2.7; footprint Resistor_SMD:R_0603_1608Metric_Pad0.98x0.95mm_HandSolder -> Resistor_SMD:R_0805_2012Metric_Pad1.20x1.40mm_HandSolder
Connections:
- net +12V: now also C3.1, C14.1, D2.2 (A), U11.5 (VCC), U4.5 (VCC), U9.5 (VCC); no longer C3.2
- net A: now also C2.2, U11.6 (VS); no longer C2.1
- net B: now also C15.2, R28.1, U4.6 (VS); no longer C4.1, R8.1
- net C: now also C4.2, R8.1, U9.6 (VS)
- net Enable: now also U11.2 (~{SD}), U4.2 (~{SD}), U9.2 (~{SD}); no longer R1.2
- net G3: now also R1.2, R28.2; no longer R6.2, R8.2
- net G4: now also R27.2, R32.2; no longer R7.2, R9.2
- net G5: now also R6.2, R8.2
- net G6: now also R7.2, R9.2
- net GND: now also C3.2, C14.2, R32.1, U11.3 (COM), U4.3 (COM), U9.3 (COM); no longer C3.1, R1.1
- net IN_A: now also U11.1 (IN)
- net IN_B: now also U4.1 (IN)
- net IN_C: now also U9.1 (IN)
- net at R2.1: now also U11.7 (HO)
- net at D1.1 (K): now also C2.1, U11.8 (VB); no longer C2.2
- net at R3.1: now also U11.4 (LO)
- net at D3.1 (K): now also C4.1, U9.8 (VB); no longer C4.2
- net at R6.1: now also U9.7 (HO)
- net at R7.1: now also U9.4 (LO)
- new net: R27.1, U4.4 (LO)
- new net: R1.1, U4.7 (HO)
- new net: C15.1, D2.1 (K), U4.8 (VB)
Other:
- moved on the sheet: C2, D1, R2, R3, R4, R5

Commit message: Добавил документы
Other:
- moved on the sheet: C1, C14, C15, C2, C3, C4, D1, D2, D3, R1, R2, R27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

Commit message: Добавил все документы
Parts:
- renumbered C14 to C2, C2 to C4, C15 to C5, C4 to C6, R4 to R1, R3 to R10, R27 to R11, R7 to R12, R28 to R2, R8 to R3, R5 to R4, R32 to R5, R9 to R6, R2 to R7, R1 to R8, R6 to R9, U11 to U1, U4 to U2, U9 to U3

Commit message: Версия под отчёт
Changed lines of the file:
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@@
   )
   (text "Драйвер С" (at 221.615 66.04 0)
-    (effects (font (size 2 2) (thickness 0.254) bold) (justify left bottom))
+    (effects (font (size 2.5 2.5) (thickness 0.254) bold) (justify left bottom))
   )
   (text "Драйвер А" (at 69.215 66.04 0)
-    (effects (font (size 2 2) (thickness 0.254) bold) (justify left bottom))
+    (effects (font (size 2.5 2.5) (thickness 0.254) bold) (justify left bottom))
   )
   (text "Драйвер В" (at 144.145 66.04 0)
-    (effects (font (size 2 2) (thickness 0.254) bold) (justify left bottom))
+    (effects (font (size 2.5 2.5) (thickness 0.254) bold) (justify left bottom))
   )
   (global_label "IN_A" (shape input) (at 55.88 107.95 180) (fields_autoplaced)

Commit message: VER2.0
Parts:
- added D10, D12, D14, D4, D5, D6: D_Small, Diode_SMD:D_SMA_Handsoldering, symbol Device:D_Small
Connections:
- net G1: now also D6.2 (A)
- net G2: now also D10.2 (A)
- net G3: now also D5.2 (A)
- net G4: now also D4.2 (A)
- net G5: now also D12.2 (A)
- net G6: now also D14.2 (A)
- net at R12.1, U3.4 (LO): now also D14.1 (K)
- net at R11.1, U2.4 (LO): now also D4.1 (K)
- net at R8.1, U2.7 (HO): now also D5.1 (K)
- net at R7.1, U1.7 (HO): now also D6.1 (K)
- net at R9.1, U3.7 (HO): now also D12.1 (K)
- net at R10.1, U1.4 (LO): now also D10.1 (K)

Commit message: Новые драйвера и разъёмы
Parts:
- removed D10, D12, D14, D4, D5, D6: D_Small, Diode_SMD:D_SMA_Handsoldering, symbol Device:D_Small
- removed U1, U2, U3: IR2184, Package_SO:SO-8_3.9x4.9mm_P1.27mm, symbol Driver_FET:IR2184
- added C25, C26, C27, C28, C29, C40: 56p, Capacitor_SMD:C_0603_1608Metric_Pad1.08x0.95mm_HandSolder, symbol Device:C_Small
- added D10, D4, D6: NSD1624, Package_SO:SOIC-8_3.9x4.9mm_P1.27mm, symbol Novosense:NSD1624
- R1, R2, R3, R4, R5, R6: value 10k -> 0
Connections:
- net +12V: now also D10.5 (VDD), D4.5 (VDD), D6.5 (VDD)
- net A: now also D6.6 (SW); no longer R1.1
- net B: now also D10.6 (SW); no longer R2.1
- net C: now also D4.6 (SW); no longer R3.1
- net G1: no longer R1.2
- net G2: no longer R4.2
- net G3: no longer R2.2
- net G4: no longer R5.2
- net G5: no longer R3.2
- net G6: no longer R6.2
- net GND: now also C25.2, C26.1, C27.1, C28.2, C29.1, C40.2, D10.3 (GND), D4.3 (GND), D6.3 (GND); no longer R4.1, R5.1, R6.1
- net at R12.1: now also D4.4 (LO)
- net at R8.1: now also D10.7 (HO)
- net at R11.1: now also D10.4 (LO)
- net at C5.1, D2.1 (K): now also D10.8 (BST)
- net at C6.1, D3.1 (K): now also D4.8 (BST)
- net at R7.1: now also D6.7 (HO)
- net at R9.1: now also D4.7 (HO)
- net at R10.1: now also D6.4 (LO)
- net at C4.1, D1.1 (K): now also D6.8 (BST)
- new net: C26.2, D6.1 (HI), R2.2
- new net: C29.2, D4.1 (HI), R5.2
- new net: C40.1, D4.2 (LI), R6.2
- new net: C25.1, D6.2 (LI), R1.2
- new net: C28.1, D10.2 (LI), R4.2
- new net: C27.2, D10.1 (HI), R3.2
- new net HI_A: R2.1
- new net HI_B: R3.1
- new net HI_C: R5.1
- new net LI_A: R1.1
- new net LI_B: R4.1
- new net LI_C: R6.1
Other:
- moved on the sheet: C1, C2, C3, C4, C5, C6, D1, D2, D3, R10, R11, R12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
