File: Плата управления/Driver.kicad_sch (KiCad schematic)
At the start: 30 parts

Commit message: Добавил все в BOM
Parts:
- D1, D2, D3: footprint Diode_SMD:D_SOD-323 -> Diode_SMD:D_SMA
Changed lines of the file:
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@@
 			)
 		)
-		(property "Footprint" "Diode_SMD:D_SOD-323"
+		(property "Footprint" "Diode_SMD:D_SMA"
 			(at 241.3 88.9 90)
 			(effects
@@
 			)
 		)
-		(property "Footprint" "Diode_SMD:D_SOD-323"
+		(property "Footprint" "Diode_SMD:D_SMA"
 			(at 163.83 88.9 90)
 			(effects
@@
 			)
 		)
-		(property "Footprint" "Diode_SMD:D_SOD-323"
+		(property "Footprint" "Diode_SMD:D_SMA"
 			(at 87.63 88.9 90)
 			(effects
